File: Mainboard/tiviaBoard.sch (KiCad schematic (older format))
At the start: 1 part, among them J1 Ti_Booster_40_J1

Commit message: Made space for TM4C123 USB connector
Other:
- note added: "LED_B"
- note added: "LED_G"
- note added: "LED_R"
Changed lines of the file:
@@
 32 A5 BE 09 BA 48 21 C5 E2 65 A5 D9 BC 20 6B 5B B8 83 64 B2 21 D0 C4 D6 7D F8 03 B3 59 26 1D 1E
 7F 93 77 53 7B B5 9A 53 C8 EA 92 4D 52 88 29 49 6C C6 A2 96 0D 0D 05 A4 F0 FF 83 88 FF 0B 96 8F
-AE AD C3 83 87 45 00 00 00 00 49 45 4E 44 AE 42 60 82 1A
+AE AD C3 83 87 45 00 00 00 00 49 45 4E 44 AE 42 60 82 00
 EndData
 $EndBitmap
@@
 61 20 10 88 FF 08 E8 4A 06 02 81 40 20 10 08 95 80 5E F5 8E 40 20 10 08 04 42 25 A0 45 06 02 81
 40 20 10 08 95 80 16 19 08 04 02 81 40 20 54 C2 FF 01 D3 55 27 F0 0D 6A 9E 83 00 00 00 00 49 45
-4E 44 AE 42 60 82 00
+4E 44 AE 42 60 82 4E
 EndData
 $EndBitmap
@@
 SSI_3_TX
 NoConn ~ 6200 1900
+Text Notes 5400 2650 0    60   ~ 0
+LED_R
+Text Notes 8350 1700 0    60   ~ 0
+LED_B
+Text Notes 8350 1800 0    60   ~ 0
+LED_G
 $EndSCHEMATC

Commit message: Still Missing WS2811 level shifter
Parts:
- removed J1: Ti_Booster_40_J1, my_foots:Tivia_Launch_Pad, symbol Ti_Booster_40_J1
- added J1: Ti_Booster_40, my_foots:Tivia_Launch_Pad, symbol Ti_Booster_40
Other:
- note added: "& (PB6)"
- note added: "& (PB7)"
- note added: "& (PD0)"
- note added: "& (PD1)"
- note added: "* Remove R10 on the launchpad evaluation board to avoid \n 2 GPIO pins connected in parallel on 2.06 and 3.04"
Changed lines of the file:
@@
 32 A5 BE 09 BA 48 21 C5 E2 65 A5 D9 BC 20 6B 5B B8 83 64 B2 21 D0 C4 D6 7D F8 03 B3 59 26 1D 1E
 7F 93 77 53 7B B5 9A 53 C8 EA 92 4D 52 88 29 49 6C C6 A2 96 0D 0D 05 A4 F0 FF 83 88 FF 0B 96 8F
-AE AD C3 83 87 45 00 00 00 00 49 45 4E 44 AE 42 60 82 00
+AE AD C3 83 87 45 00 00 00 00 49 45 4E 44 AE 42 60 82 FF
 EndData
 $EndBitmap
@@
 61 20 10 88 FF 08 E8 4A 06 02 81 40 20 10 08 95 80 5E F5 8E 40 20 10 08 04 42 25 A0 45 06 02 81
 40 20 10 08 95 80 16 19 08 04 02 81 40 20 54 C2 FF 01 D3 55 27 F0 0D 6A 9E 83 00 00 00 00 49 45
-4E 44 AE 42 60 82 4E
+4E 44 AE 42 60 82 00
 EndData
 $EndBitmap
@@
 Wire Wire Line
 	1650 1800 1650 1800
-$Comp
-L Ti_Booster_40_J1 J1
-U 1 1 566EC104
-P 1600 2800
-F 0 "J1" H 2200 4100 60  0000 C CNN
-F 1 "Ti_Booster_40_J1" H 2250 2800 60  0000 C CNN
-F 2 "my_foots:Tivia_Launch_Pad" H 2250 3450 60  0001 C CNN
-F 3 "" H 2250 3450 60  0000 C CNN
-	1    1600 2800
-	1    0    0    -1
-$EndComp
-$Comp
-L Ti_Booster_40_J1 J1
-U 3 1 566EC105
-P 6150 2800
-F 0 "J1" H 6750 4100 60  0000 C CNN
-F 1 "Ti_Booster_40_J1" H 6800 2800 60  0000 C CNN
-F 2 "my_foots:Tivia_Launch_Pad" H 6800 3450 60  0001 C CNN
-F 3 "" H 6800 3450 60  0000 C CNN
-	3    6150 2800
-	1    0    0    -1
-$EndComp
-$Comp
-L Ti_Booster_40_J1 J1
-U 4 1 566EC106
-P 8650 2800
-F 0 "J1" H 9250 4100 60  0000 C CNN
-F 1 "Ti_Booster_40_J1" H 9300 2800 60  0000 C CNN
-F 2 "my_foots:Tivia_Launch_Pad" H 9300 3450 60  0001 C CNN
-F 3 "" H 9300 3450 60  0000 C CNN
-	4    8650 2800
-	1    0    0    -1
-$EndComp
-$Comp
-L Ti_Booster_40_J1 J1
-U 2 1 566EC107
-P 3750 2800
-F 0 "J1" H 4350 4100 60  0000 C CNN
-F 1 "Ti_Booster_40_J1" H 4400 2800 60  0000 C CNN
-F 2 "my_foots:Tivia_Launch_Pad" H 4400 3450 60  0001 C CNN
-F 3 "" H 4400 3450 60  0000 C CNN
-	2    3750 2800
-	1    0    0    -1
-$EndComp
 Text HLabel 1650 1800 0    60   Output ~ 0
 po_3_pwm
@@
 Text HLabel 1650 2600 0    60   BiDi ~ 0
 I2C1_SDA
-Text HLabel 3800 2300 0    60   BiDi ~ 0
+Text HLabel 6200 1900 0    60   BiDi ~ 0
 I2C3_SCL
-Text HLabel 3800 2200 0    60   BiDi ~ 0
+Text HLabel 6200 2000 0    60   BiDi ~ 0
 ISC3_SDA
 Text HLabel 8700 2400 0    60   Input ~ 0
@@
 NoConn ~ 8700 1700
 NoConn ~ 8700 1800
-$Comp
-L PWR_FLAG #FLG054
-U 1 1 56751E81
-P 1250 1200
-F 0 "#FLG054" H 1250 1295 50  0001 C CNN
-F 1 "PWR_FLAG" H 1250 1380 50  0000 C CNN
-F 2 "" H 1250 1200 50  0000 C CNN
-F 3 "" H 1250 1200 50  0000 C CNN
-	1    1250 1200
-	-1   0    0    1
-$EndComp
-Connection ~ 1250 1200
 Text HLabel 3800 2600 0    60   Output ~ 0
 SSI_0_CLK
@@
 Text HLabel 3800 2500 0    60   Output ~ 0
 SSI_0_/SS
-Text HLabel 6200 2000 0    60   Output ~ 0
+Text HLabel 3800 2200 0    60   Output ~ 0
 SSI_2_TX
 Text HLabel 6200 2200 0    60   Output ~ 0
 SSI_3_TX
-NoConn ~ 6200 1900
 Text Notes 5400 2650 0    60   ~ 0
 LED_R
@@
 Text Notes 8350 1800 0    60   ~ 0
 LED_G
+Text Notes 4500 2250 0    60   ~ 0
+& (PD1)
+Text Notes 4500 2350 0    60   ~ 0
+& (PD0)
+Text Notes 6900 1950 0    60   ~ 0
+& (PB6)
+Text Notes 6900 2050 0    60   ~ 0
+& (PB7)
+Text Notes 7100 6750 0    60   ~ 0
+* Remove R10 on the launchpad evaluation board to avoid \n   2 GPIO pins connected in parallel on 2.06 and 3.04
+NoConn ~ 3800 2300
+$Comp
+L Ti_Booster_40 J1
+U 1 1 5691947B
+P 1600 2800
+F 0 "J1" H 2200 4100 60  0000 C CNN
+F 1 "Ti_Booster_40" H 2250 2800 60  0000 C CNN
+F 2 "my_foots:Tivia_Launch_Pad" H 2250 3450 60  0001 C CNN
+F 3 "" H 2250 3450 60  0000 C CNN
+	1    1600 2800
+	1    0    0    -1
+$EndComp
+$Comp
+L Ti_Booster_40 J1
+U 2 1 569194AC
+P 3750 2800
+F 0 "J1" H 4350 4100 60  0000 C CNN
+F 1 "Ti_Booster_40" H 4400 2800 60  0000 C CNN
+F 2 "my_foots:Tivia_Launch_Pad" H 4400 3450 60  0001 C CNN
+F 3 "" H 4400 3450 60  0000 C CNN
+	2    3750 2800
+	1    0    0    -1
+$EndComp
+$Comp
+L Ti_Booster_40 J1
+U 3 1 569194E5
+P 6150 2800
+F 0 "J1" H 6750 4100 60  0000 C CNN
+F 1 "Ti_Booster_40" H 6800 2800 60  0000 C CNN
+F 2 "my_foots:Tivia_Launch_Pad" H 6800 3450 60  0001 C CNN
+F 3 "" H 6800 3450 60  0000 C CNN
+	3    6150 2800
+	1    0    0    -1
+$EndComp
+$Comp
+L Ti_Booster_40 J1
+U 4 1 56919524
+P 8650 2800
+F 0 "J1" H 9250 4100 60  0000 C CNN
+F 1 "Ti_Booster_40" H 9300 2800 60  0000 C CNN
+F 2 "my_foots:Tivia_Launch_Pad" H 9300 3450 60  0001 C CNN
+F 3 "" H 9300 3450 60  0000 C CNN
+	4    8650 2800
+	1    0    0    -1
+$EndComp
 $EndSCHEMATC
