File: Mainboard/fan_tas_tic.sch (KiCad schematic (older format))
At the start: 82 parts, among them P1 CONN_01X04, P10 CONN_01X08, P11 CONN_01X04, P12 CONN_01X04, P13 CONN_01X04, P14 CONN_01X04, P2 CONN_01X04, P3 CONN_01X04, P4 CONN_01X04, P5 CONN_01X04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

Commit message: Small documentation updates
Other:
- note added: "Blue\nWhite\nYellow\nGreen\nPurple\nBlack\nBrown\nOrange"
- note added: "Row In\n(Black shrink wrap on cable)"
- note added: "Row\n(cable with no shrink wrap)"
- note removed: "Row In"
Changed lines of the file:
@@
 	1    0    0    -1
 $EndComp
-Text Notes 10350 9500 0    60   ~ 0
+Text Notes 8800 8400 0    60   ~ 0
 Row Out\ndrive only one of the outputs low\nInit: keep Ser_In and RCK low, pulse SRCK 8 times\nEnable Drain0:  keep Ser_in and RCK high, pulse SRCK, pulse Ser_in and RCK\n      ...  from now on, keep Ser_in and RCK low ...\nEnable Drain1:  pulse SRCK, pulse Ser_in and RCK
-Text Notes 9850 4600 0    60   ~ 0
-Row In
+Text Notes 10200 4650 0    60   ~ 0
+Row In\n(Black shrink wrap on cable)
 $Comp
 L CONN_01X08 P7
@@
 Connection ~ 3850 2800
 Connection ~ 3050 1450
+Text Notes 10200 5500 0    60   ~ 0
+Blue\nWhite\nYellow\nGreen\nPurple\nBlack\nBrown\nOrange
+Text Notes 10100 9650 0    60   ~ 0
+Blue\nWhite\nYellow\nGreen\nPurple\nBlack\nBrown\nOrange
+Text Notes 10100 8850 0    60   ~ 0
+Row\n(cable with no shrink wrap)
 $EndSCHEMATC
