File: Mainboard/fan_tas_tic.kicad_pcb (KiCad board)
At the start: 2 copper layers, 155 x 175 mm, 127 parts, among them J1 Ti_Booster_40, P1 CONN_01X04, P10 CONN_01X08, P11 CONN_01X04, P12 CONN_01X04, P13 CONN_01X04, P14 CONN_01X04, P2 CONN_01X04, P3 CONN_01X04, P4 CONN_01X04, P5 CONN_01X04, P6 CONN_01X08, P7 CONN_01X08, P8 CONN_01X08, P9 CONN_01X08, Q1 IRL640, Q10 IRL640, Q11 IRL640, Q12 IRL640, Q13 BSS138, Q14 BSS138, Q15 BSS138, Q16 BSS138, Q17 BSS138, Q18 BSS138, Q19 BSS138, Q2 IRL640, Q20 BSS138, Q3 IRL640, Q4 IRL640, Q5 IRL640, Q6 IRL640, Q7 IRL640, Q8 IRL640, Q9 IRL640, U1 7812, U2 7805, U3 UCC27524, U4 UCC27524, U5 TPIC6B595, U6 PCF8574, U7 74HC04

Commit message: Updated Schematic with minor changes after first prototype
Parts:
- added D10: 1N5822, Diodes_ThroughHole:Diode_DO-201AD_Horizontal_RM15, F.Cu at (80.0, 244.8)
- added D11: 1N5822, Diodes_ThroughHole:Diode_DO-201AD_Horizontal_RM15, F.Cu at (92.5, 245.0)
- added D12: 1N5822, Diodes_ThroughHole:Diode_DO-201AD_Horizontal_RM15, F.Cu at (105.0, 244.8)
- added D13: 1N5822, Diodes_ThroughHole:Diode_DO-201AD_Horizontal_RM15, F.Cu at (117.5, 244.8)
- added D14: 1N5822, Diodes_ThroughHole:Diode_DO-201AD_Horizontal_RM15, F.Cu at (130.0, 244.8)
- added D15: 1N5822, Diodes_ThroughHole:Diode_DO-201AD_Horizontal_RM15, F.Cu at (142.5, 244.8)
- added D16: 1N5822, Diodes_ThroughHole:Diode_DO-201AD_Horizontal_RM15, F.Cu at (155.0, 244.8)
- added D4: D_Schottky, Diodes_ThroughHole:Diode_DO-201AD_Horizontal_RM15, F.Cu at (5.00, 244.8)
- added D5: 1N5822, Diodes_ThroughHole:Diode_DO-201AD_Horizontal_RM15, F.Cu at (17.5, 244.8)
- added D6: 1N5822, Diodes_ThroughHole:Diode_DO-201AD_Horizontal_RM15, F.Cu at (30.0, 245.0)
- added D7: 1N5822, Diodes_ThroughHole:Diode_DO-201AD_Horizontal_RM15, F.Cu at (42.5, 244.8)
- added D8: 1N5822, Diodes_ThroughHole:Diode_DO-201AD_Horizontal_RM15, F.Cu at (55.0, 244.8)
- added D9: 1N5822, Diodes_ThroughHole:Diode_DO-201AD_Horizontal_RM15, F.Cu at (67.5, 245.0)
- added JP2: Jumper_NO_Small, Pin_Headers:Pin_Header_Straight_1x02, F.Cu at (74.3, 41.9)
- added K1: RELAY_2RT, Relays_ThroughHole:Relay_DPDT_Schrack-RT2_RM5mm, F.Cu at (-5.00, 222.5)
- added Q21: BSS138, TO_SOT_Packages_SMD:SOT-23, F.Cu at (-5.95, 207.5)
- added R47: 4k7, Resistors_ThroughHole:Resistor_Vertical_RM5mm, F.Cu at (-12.5, 205.0)
- R1, R14, R2, R5: value 47R -> 200R
- moved RR1 1.26 mm to (40.6, 48.9)
Connections:
- C1 pad 1: +24V -> Net-(C1-Pad1)
- J1 pad 13: Net-(J1-Pad13) -> /TiviaBoard/PE0_24V_ENABLE
- J1 pad 14: Net-(J1-Pad14) -> (no net)
- J1 pad 15: Net-(J1-Pad15) -> (no net)
- J1 pad 17: Net-(J1-Pad17) -> (no net)
- J1 pad 18: /TiviaBoard/SSI_0_RX -> (no net)
- J1 pad 19: /TiviaBoard/SSI_0_/SS -> (no net)
- J1 pad 20: /TiviaBoard/SSI_0_CLK -> (no net)
- J1 pad 25: Net-(J1-Pad25) -> (no net)
- J1 pad 31: Net-(J1-Pad31) -> (no net)
- J1 pad 32: Net-(J1-Pad32) -> (no net)
- J1 pad 8: /TiviaBoard/SSI_0_TX -> (no net)
- P1 pad 3: +24V -> Net-(C1-Pad1)
- P1 pad 4: +24V -> Net-(C1-Pad1)
- U1 pad VI: +24V -> Net-(C1-Pad1)
- U5 pad 1: Net-(U5-Pad1) -> (no net)
- U5 pad 18: Net-(U5-Pad18) -> (no net)
- U5 pad 20: Net-(U5-Pad20) -> (no net)
- U6 pad 13: Net-(U6-Pad13) -> (no net)
Routing:
- net +24V: track 251.7 -> 232.7 mm
- net Net-(C1-Pad1): track 0.00 -> 19.0 mm
- net +5V: track 512.9 -> 527.5 mm
- net /I2C_LEVEL_SHIFT2/B_3V3: track 60.7 -> 68.7 mm
- net /I2C_LEVEL_SHIFT1/B_3V3: track 119.9 -> 126.7 mm
- net /I2C_LEVEL_SHIFT2/A_3V3: track 58.7 -> 65.3 mm
- net /I2C_LEVEL_SHIFT1/A_3V3: track 108.2 -> 114.3 mm
- net +5VP: track 106.6 -> 110.7 mm
- net /TiviaBoard/SSI_3_TX: track 52.1 -> 56.0 mm
- net +3V3: track 341.2 -> 343.7 mm
- net Net-(R51-Pad2): track 22.2 -> 23.8 mm
- net +12V: track 204.9 -> 203.9 mm
Other:
- board text added: "06/2016"
- board text added: "1.1"
- board text added: "ToDo list: * Move USB DEBUG out of the way! (crashes with I2C extension ports) * Add more decoupling caps! * Add Schottky freewheeling diodes * Add 24V relay circuit"
- board text removed: "01/2016"
- board text removed: "1.0"
