File: Mainboard/fan_tas_tic.kicad_pcb (KiCad board)
At the start: 2 copper layers, 155 x 175 mm, 151 parts, among them J1 Ti_Booster_40, K1 RELAY_2RT, P1 CONN_01X04, P10 CONN_01X08, P11 CONN_01X04, P12 CONN_01X04, P13 CONN_01X04, P14 CONN_01X04, P2 CONN_01X04, P3 CONN_01X04, P4 CONN_01X04, P5 CONN_01X04, P6 CONN_01X08, P7 CONN_01X08, P8 CONN_01X08, P9 CONN_01X08, Q1 IRL640, Q10 IRL640, Q11 IRL640, Q12 IRL640, Q13 BSS138, Q14 BSS138, Q15 BSS138, Q16 BSS138, Q17 BSS138, Q18 BSS138, Q19 BSS138, Q2 IRL640, Q20 BSS138, Q21 BSS138, Q3 IRL640, Q4 IRL640, Q5 IRL640, Q6 IRL640, Q7 IRL640, Q8 IRL640, Q9 IRL640, U1 7812, U2 7805, U3 UCC27524, U4 UCC27524, U5 TPIC6B595, U6 PCF8574, U7 74HC04

Commit message: Added 8 additional Mosfet channels, cleaned up rouing a bit
Parts:
- added C33: 470nF, Capacitors_SMD:C_0805_HandSoldering, F.Cu at (101.6, 98.4)
- added C34: 470nF, Capacitors_SMD:C_0805_HandSoldering, F.Cu at (101.6, 106.0)
- added C35: 470nF, Capacitors_SMD:C_0805_HandSoldering, F.Cu at (101.6, 113.7)
- added C36: 470nF, Capacitors_SMD:C_0805_HandSoldering, F.Cu at (101.6, 120.7)
- added C37: 470nF, Capacitors_SMD:C_0805_HandSoldering, F.Cu at (101.6, 142.9)
- added C38: 470nF, Capacitors_SMD:C_0805_HandSoldering, F.Cu at (101.6, 150.6)
- added C39: 470nF, Capacitors_SMD:C_0805_HandSoldering, F.Cu at (101.6, 158.1)
- added C40: 470nF, Capacitors_SMD:C_0805_HandSoldering, F.Cu at (101.6, 166.4)
- added C41: 470 nF, Capacitors_SMD:C_0805_HandSoldering, F.Cu at (99.8, 132.1)
- added C43: 4700 uF, 30 V, Capacitors_ThroughHole:C_Radial_D18_L36_P7.5, F.Cu at (109.5, 86.9)
- added C44: 4700 uF, 30 V, Capacitors_ThroughHole:C_Radial_D18_L36_P7.5, F.Cu at (128.3, 175.3)
- added C45: 4700 uF, 30 V, Capacitors_ThroughHole:C_Radial_D14_L25_P5, F.Cu at (159.5, 85.6)
- added C46: 4700 uF, 30 V, Capacitors_ThroughHole:C_Radial_D14_L25_P5, F.Cu at (118.4, 129.8)
- added D16: SS34, Diodes_SMD:SMC-RM10_Universal_Handsoldering, F.Cu at (118.1, 98.5)
- added D17: SS34, Diodes_SMD:SMC-RM10_Universal_Handsoldering, F.Cu at (118.2, 106.1)
- added D18: SS34, Diodes_SMD:SMC-RM10_Universal_Handsoldering, F.Cu at (118.0, 113.7)
- added D19: SS34, Diodes_SMD:SMC-RM10_Universal_Handsoldering, F.Cu at (118.2, 121.3)
- added D20: SS34, Diodes_SMD:SMC-RM10_Universal_Handsoldering, F.Cu at (118.1, 143.5)
- added D21: SS34, Diodes_SMD:SMC-RM10_Universal_Handsoldering, F.Cu at (118.0, 151.1)
- added D22: SS34, Diodes_SMD:SMC-RM10_Universal_Handsoldering, F.Cu at (118.1, 158.8)
- added D23: SS34, Diodes_SMD:SMC-RM10_Universal_Handsoldering, F.Cu at (118.0, 166.4)
- added P11: CONN_01X08, my_foots:HT396_8, F.Cu at (102.7, 96.1)
- added P12: CONN_01X08, my_foots:HT396_8, F.Cu at (102.7, 141.0)
- added Q13: IRL640, TO_SOT_Packages_THT:TO-220_Neutral123_Vertical_LargePads, F.Cu at (96.5, 98.5)
- added Q14: IRL640, TO_SOT_Packages_THT:TO-220_Neutral123_Vertical_LargePads, F.Cu at (96.5, 106.1)
- added Q15: IRL640, TO_SOT_Packages_THT:TO-220_Neutral123_Vertical_LargePads, F.Cu at (96.5, 113.7)
- added Q16: IRL640, TO_SOT_Packages_THT:TO-220_Neutral123_Vertical_LargePads, F.Cu at (96.5, 121.3)
- added Q17: IRL640, TO_SOT_Packages_THT:TO-220_Neutral123_Vertical_LargePads, F.Cu at (96.5, 143.5)
- added Q18: IRL640, TO_SOT_Packages_THT:TO-220_Neutral123_Vertical_LargePads, F.Cu at (96.5, 151.1)
- added Q19: IRL640, TO_SOT_Packages_THT:TO-220_Neutral123_Vertical_LargePads, F.Cu at (96.5, 158.8)
- added Q20: IRL640, TO_SOT_Packages_THT:TO-220_Neutral123_Vertical_LargePads, F.Cu at (96.5, 166.4)
- added R49: 470R, Resistors_SMD:R_0805_HandSoldering, F.Cu at (88.9, 98.5)
- added R50: 470R, Resistors_SMD:R_0805_HandSoldering, F.Cu at (88.9, 106.2)
- added R52: 470R, Resistors_SMD:R_0805_HandSoldering, F.Cu at (88.9, 121.2)
- added R53: 470R, Resistors_SMD:R_0805_HandSoldering, F.Cu at (88.9, 143.5)
- added R54: 470R, Resistors_SMD:R_0805_HandSoldering, F.Cu at (88.9, 151.1)
- added R55: 470R, Resistors_SMD:R_0805_HandSoldering, F.Cu at (88.9, 158.8)
- added R56: 470R, Resistors_SMD:R_0805_HandSoldering, F.Cu at (88.9, 166.4)
- added R57: 470, Resistors_SMD:R_0805_HandSoldering, F.Cu at (73.6, 31.8)
- added U7: PCF8574, Housings_SOIC:SOIC-16_7.5x10.3mm_Pitch1.27mm, F.Cu at (92.7, 132.1)
- C10, C12, C14, C15, C21, C22, C25, C26, C27, C28, C29, C30, C31, C32, C5, C6, C7, C8, C9, F4, R10, R11, R12, R13, R33, R37, R41, R45, R6, R7, R8, R9: moved to F.Cu
- C42: renamed from C33; moved to F.Cu
- R51: value 470 -> 470R; footprint Resistors_ThroughHole:Resistor_Vertical_RM5mm -> Resistors_SMD:R_0805_HandSoldering
- moved C2 274.7 mm to (93.3, 24.1), turned to 270 degrees
- moved R47 187.1 mm to (116.8, 47.0), turned to 0 degrees
- moved R48 176.8 mm to (122.6, 50.2), turned to 180 degrees
- moved C24 173.7 mm to (82.6, 62.9)
- moved Q21 171.9 mm to (122.6, 47.0)
- moved R51 80.3 mm to (88.9, 113.8), turned to 270 degrees
- moved R19 63.6 mm to (22.2, 99.1), turned to 90 degrees
- moved P6 45.0 mm to (47.2, 179.7), turned to 90 degrees
- moved C16 31.6 mm to (74.9, 41.9), turned to 270 degrees
- moved F5 29.7 mm to (104.1, 33.0), turned to 270 degrees
- moved D25 29.2 mm to (91.4, 40.6), turned to 180 degrees
- moved C23 24.7 mm to (64.1, 39.4), turned to 270 degrees
- moved U4 23.3 mm to (118.1, 69.8)
- moved C11 22.9 mm to (53.6, 160.7), turned to 180 degrees
- moved C19 22.2 mm to (53.6, 156.8), turned to 180 degrees
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- renumbered D13 to D12, D14 to D13, D15 to D14, D16 to D15, D12 to D24, D17 to D25, P12 to P15, P11 to P16, Q13 to Q22, Q14 to Q23, Q15 to Q24, Q16 to Q25, Q17 to Q26, Q18 to Q27, Q19 to Q28, Q20 to Q29, U7 to U8
Connections:
- J1 pad 14: (no net) -> Net-(J1-Pad14)
- J1 pad 15: (no net) -> Net-(J1-Pad15)
- J1 pad 17: (no net) -> Net-(J1-Pad17)
- J1 pad 18: (no net) -> /TiviaBoard/SSI_0_RX
- J1 pad 19: (no net) -> /TiviaBoard/SSI_0_/SS
- J1 pad 20: (no net) -> /TiviaBoard/SSI_0_CLK
- J1 pad 25: (no net) -> Net-(J1-Pad25)
- J1 pad 31: (no net) -> Net-(J1-Pad31)
- J1 pad 32: (no net) -> Net-(J1-Pad32)
- J1 pad 8: (no net) -> /TiviaBoard/SSI_0_TX
- K1 pad 14: (no net) -> Net-(K1-Pad14)
- K1 pad 3: (no net) -> Net-(K1-Pad3)
- R51 pad 1: Net-(P13-Pad3) -> Net-(Q15-Pad1)
- R51 pad 2: Net-(R51-Pad2) -> /powerChannel10/CTRL
- U5 pad 1: (no net) -> Net-(U5-Pad1)
- U5 pad 18: (no net) -> Net-(U5-Pad18)
- U5 pad 20: (no net) -> Net-(U5-Pad20)
- U6 pad 13: (no net) -> Net-(U6-Pad13)
- U8 pad 12: Net-(R51-Pad2) -> Net-(R57-Pad2)
Routing:
- net +24V: track 300.4 -> 568.6 mm, vias 2 -> 11
- net GND: track 881.9 -> 642.5 mm, vias 7 -> 12
- net +12V: track 203.9 -> 15.6 mm
- net +3V3: track 229.7 -> 53.7 mm, vias 3 -> 0
- net /TiviaBoard/po_6_pwm: track 104.1 -> 0.00 mm, vias 1 -> 0
- net /I2C_LEVEL_SHIFT3/A_3V3: track 105.7 -> 3.11 mm
- net /TiviaBoard/po_7_pwm: track 100.8 -> 0.00 mm, vias 1 -> 0
- net /TiviaBoard/SSI_2_TX: track 100.1 -> 0.00 mm
- net +5V: track 221.7 -> 146.0 mm, vias 2 -> 4
- net /I2C_LEVEL_SHIFT1/A_3V3: track 78.7 -> 3.11 mm, vias 2 -> 0
- net /I2C_LEVEL_SHIFT2/A_3V3: track 78.0 -> 3.11 mm, vias 2 -> 0
- net /I2C_LEVEL_SHIFT3/B_3V3: track 71.3 -> 3.11 mm
- net /TiviaBoard/SSI_3_TX: track 56.0 -> 0.00 mm, vias 3 -> 0
- net /TiviaBoard/po_3_pwm: track 55.7 -> 0.00 mm, vias 1 -> 0
- net /I2C_LEVEL_SHIFT2/B_3V3: track 56.8 -> 3.11 mm, vias 2 -> 0
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Other:
- board text added: "2.0"
- board text removed: "1.1"
