File: Mainboard/powerRails.sch (KiCad schematic (older format))
At the start: 27 parts, among them K1 RELAY_2RT, P1 CONN_01X04, P11 CONN_01X04, Q21 BSS138, U1 7812, U2 7805

Commit message: Added 8 additional Mosfet channels, cleaned up rouing a bit
Parts:
- renumbered D12 to D24, D17 to D25, P11 to P16
Changed lines of the file:
@@
 $Descr A4 11693 8268
 encoding utf-8
-Sheet 8 19
+Sheet 8 27
 Title ""
 Date ""
@@
 $EndDescr
 $Comp
-L GND #PWR048
+L GND #PWR053
 U 1 1 576FCD00
 P 4300 2250
-F 0 "#PWR048" H 4300 2000 50  0001 C CNN
+F 0 "#PWR053" H 4300 2000 50  0001 C CNN
 F 1 "GND" H 4300 2100 50  0000 C CNN
 F 2 "" H 4300 2250 50  0000 C CNN
@@
 $EndComp
 $Comp
-L +24V #PWR049
+L +24V #PWR054
 U 1 1 576FCD03
 P 5350 3050
-F 0 "#PWR049" H 5350 2900 50  0001 C CNN
+F 0 "#PWR054" H 5350 2900 50  0001 C CNN
 F 1 "+24V" H 5350 3190 50  0000 C CNN
 F 2 "" H 5350 3050 50  0000 C CNN
@@
 $EndComp
 $Comp
-L +12V #PWR050
+L +12V #PWR055
 U 1 1 576FCD04
 P 4700 1850
-F 0 "#PWR050" H 4700 1700 50  0001 C CNN
+F 0 "#PWR055" H 4700 1700 50  0001 C CNN
 F 1 "+12V" H 4700 1990 50  0000 C CNN
 F 2 "" H 4700 1850 50  0000 C CNN
@@
 $EndComp
 $Comp
-L GND #PWR051
+L GND #PWR056
 U 1 1 576FCD07
 P 6700 2250
-F 0 "#PWR051" H 6700 2000 50  0001 C CNN
+F 0 "#PWR056" H 6700 2000 50  0001 C CNN
 F 1 "GND" H 6700 2100 50  0000 C CNN
 F 2 "" H 6700 2250 50  0000 C CNN
@@
 $EndComp
 $Comp
-L +5V #PWR052
+L +5V #PWR057
 U 1 1 576FCD4C
 P 7550 1850
-F 0 "#PWR052" H 7550 1700 50  0001 C CNN
+F 0 "#PWR057" H 7550 1700 50  0001 C CNN
 F 1 "+5V" H 7550 1990 50  0000 C CNN
 F 2 "" H 7550 1850 50  0000 C CNN
@@
 +5V can come from:\n  * USB (leave both jumpers open)\n  * LED supply (close JP2)\n  * 24 V solenoid supply (close JP1)
 $Comp
-L CONN_01X04 P11
+L CONN_01X04 P16
 U 1 1 576FCD4E
 P 3050 7000
-F 0 "P11" H 3050 7250 50  0000 C CNN
+F 0 "P16" H 3050 7250 50  0000 C CNN
 F 1 "CONN_01X04" V 3150 7000 50  0000 C CNN
 F 2 "my_foots:HT396_4" H 3050 7000 50  0001 C CNN
@@
 $EndComp
 $Comp
-L GND #PWR053
+L GND #PWR058
 U 1 1 576FCD51
 P 3550 7150
-F 0 "#PWR053" H 3550 6900 50  0001 C CNN
+F 0 "#PWR058" H 3550 6900 50  0001 C CNN
 F 1 "GND" H 3550 7000 50  0000 C CNN
 F 2 "" H 3550 7150 50  0000 C CNN
@@
 $EndComp
 $Comp
-L PWR_FLAG #FLG054
+L PWR_FLAG #FLG059
 U 1 1 576FCD58
 P 2300 1850
-F 0 "#FLG054" H 2300 1945 50  0001 C CNN
+F 0 "#FLG059" H 2300 1945 50  0001 C CNN
 F 1 "PWR_FLAG" H 2300 2030 50  0000 C CNN
 F 2 "" H 2300 1850 50  0000 C CNN
@@
 $EndComp
 $Comp
-L PWR_FLAG #FLG055
+L PWR_FLAG #FLG060
 U 1 1 576FCD59
 P 3900 6850
-F 0 "#FLG055" H 3900 6945 50  0001 C CNN
+F 0 "#FLG060" H 3900 6945 50  0001 C CNN
 F 1 "PWR_FLAG" H 3900 7030 50  0000 C CNN
 F 2 "" H 3900 6850 50  0000 C CNN
@@
 $EndComp
 $Comp
-L GND #PWR056
+L GND #PWR061
 U 1 1 576FCD6A
 P 1750 7350
-F 0 "#PWR056" H 1750 7100 50  0001 C CNN
+F 0 "#PWR061" H 1750 7100 50  0001 C CNN
 F 1 "GND" H 1750 7200 50  0000 C CNN
 F 2 "" H 1750 7350 50  0000 C CNN
@@
 $EndComp
 $Comp
-L +24V #PWR057
+L +24V #PWR062
 U 1 1 576FCD6F
 P 1050 6550
-F 0 "#PWR057" H 1050 6400 50  0001 C CNN
+F 0 "#PWR062" H 1050 6400 50  0001 C CNN
 F 1 "+24V" H 1050 6690 50  0000 C CNN
 F 2 "" H 1050 6550 50  0000 C CNN
@@
 $EndComp
 $Comp
-L +12V #PWR058
+L +12V #PWR063
 U 1 1 576FCD70
 P 1050 6800
-F 0 "#PWR058" H 1050 6650 50  0001 C CNN
+F 0 "#PWR063" H 1050 6650 50  0001 C CNN
 F 1 "+12V" H 1050 6940 50  0000 C CNN
 F 2 "" H 1050 6800 50  0000 C CNN
@@
 $EndComp
 $Comp
-L +5V #PWR059
+L +5V #PWR064
 U 1 1 576FCD71
 P 1050 7050
-F 0 "#PWR059" H 1050 6900 50  0001 C CNN
+F 0 "#PWR064" H 1050 6900 50  0001 C CNN
 F 1 "+5V" H 1050 7190 50  0000 C CNN
 F 2 "" H 1050 7050 50  0000 C CNN
@@
 $EndComp
 $Comp
-L +5VP #PWR060
+L +5VP #PWR065
 U 1 1 576FCD82
 P 4200 6850
-F 0 "#PWR060" H 4200 6700 50  0001 C CNN
+F 0 "#PWR065" H 4200 6700 50  0001 C CNN
 F 1 "+5VP" H 4200 6990 50  0000 C CNN
 F 2 "" H 4200 6850 50  0000 C CNN
@@
 $EndComp
 $Comp
-L +5V #PWR061
+L +5V #PWR066
 U 1 1 576FCD97
 P 5100 6850
-F 0 "#PWR061" H 5100 6700 50  0001 C CNN
+F 0 "#PWR066" H 5100 6700 50  0001 C CNN
 F 1 "+5V" H 5100 6990 50  0000 C CNN
 F 2 "" H 5100 6850 50  0000 C CNN
@@
 $EndComp
 $Comp
-L GND #PWR062
+L GND #PWR067
 U 1 1 576FCD9F
 P 2550 5050
-F 0 "#PWR062" H 2550 4800 50  0001 C CNN
+F 0 "#PWR067" H 2550 4800 50  0001 C CNN
 F 1 "GND" H 2550 4900 50  0000 C CNN
 F 2 "" H 2550 5050 50  0000 C CNN
@@
 Connection ~ 4000 3100
 $Comp
-L D_Schottky D17
+L D_Schottky D25
 U 1 1 577011AD
 P 4600 6850
-F 0 "D17" H 4600 6950 50  0000 C CNN
+F 0 "D25" H 4600 6950 50  0000 C CNN
 F 1 "SS34" H 4600 6750 50  0000 C CNN
 F 2 "Diodes_SMD:SMC-RM10_Universal_Handsoldering" H 4600 6850 50  0001 C CNN
@@
 	1500 4650 1850 4650
 $Comp
-L PWR_FLAG #FLG063
+L PWR_FLAG #FLG068
 U 1 1 5771DC49
 P 7850 1850
-F 0 "#FLG063" H 7850 1945 50  0001 C CNN
+F 0 "#FLG068" H 7850 1945 50  0001 C CNN
 F 1 "PWR_FLAG" H 7850 2030 50  0000 C CNN
 F 2 "" H 7850 1850 50  0000 C CNN
@@
 Connection ~ 4200 7150
 $Comp
-L D_Schottky D12
+L D_Schottky D24
 U 1 1 57721022
 P 2550 4100
-F 0 "D12" H 2550 4200 50  0000 C CNN
+F 0 "D24" H 2550 4200 50  0000 C CNN
 F 1 "SS34" H 2550 4000 50  0000 C CNN
 F 2 "Diodes_SMD:SMC-RM10_Universal_Handsoldering" H 2550 4100 50  0001 C CNN
@@
 Wire Wire Line
 	1450 1850 1200 1850
+$Comp
+L PWR_FLAG #FLG069
+U 1 1 57936202
+P 2300 2200
+F 0 "#FLG069" H 2300 2295 50  0001 C CNN
+F 1 "PWR_FLAG" H 2300 2380 50  0000 C CNN
+F 2 "" H 2300 2200 50  0000 C CNN
+F 3 "" H 2300 2200 50  0000 C CNN
+	1    2300 2200
+	1    0    0    -1
+$EndComp
+Connection ~ 2300 2200
 $EndSCHEMATC
